File: GameBox.kicad_sch (KiCad schematic)
At the start: 18 parts, among them J1 OLED, SW1 SW_down, SW2 SW_up, SW3 SW_right, SW4 SW_left, SW5 SW_select, U1 ATmega328P-P, Y1 16MHz

Commit message: Component placement
Parts:
- removed SW5: SW_select, Button_Switch_THT:SW_PUSH_6mm_H9.5mm, symbol Switch:SW_Push
- added SW1: ON/OFF, GameBox:SS12D10, symbol Switch:SW_Push_SPDT
- renumbered R3 to R1, R1 to R3, SW1 to SW2, SW2 to SW3, SW3 to SW4, SW4 to SW5
Connections:
- net VDD: now also SW1.3 (C); no longer C1.1, U1.20 (AVCC), U1.7 (VCC)
- new net: C1.1, SW1.2 (B), U1.20 (AVCC), U1.7 (VCC)
- no-connect marks 9 -> 11
Other:
- moved on the sheet: BT1, BT2
